Commit message: Few .xacro fixes

File: src/line_follower_description/urdf/dummy_bot.urdf.xacro (robot description, xacro)
@@ -1,82 +1,141 @@
 <?xml version="1.0"?>
-<robot xmlns:xacro="http://www.ros.org/wiki/xacro" name="dummy_bot">
+<robot name="my_robot" xmlns:xacro="http://www.ros.org/wiki/xacro">
+    <material name="green">
+        <color rgba="0 0.6 0 1" />
+    </material>
+    <material name="gray">
+        <color rgba="0.7 0.7 0.7 1" />
+    </material>
+    <xacro:macro name="box_inertia" params="m x y z o_xyz o_rpy">
+        <inertial>
+            <mass value="${m}" />
+            <origin xyz="${o_xyz}" rpy="${o_rpy}" />
+            <inertia ixx="${(m/12) * (z*z + y*y)}" ixy="0" ixz="0"
+                    iyy="${(m/12) * (x*x + z*z)}" iyz="0"
+                    izz="${(m/12) * (x*x + y*y)}" />
+        </inertial>
+    </xacro:macro>
+    <xacro:macro name="cylinder_inertia" params="m r l o_xyz o_rpy">
+        <inertial>
+            <mass value="${m}" />
+            <origin xyz="${o_xyz}" rpy="${o_rpy}" />
+            <inertia ixx="${(m/12) * (3*r*r + l*l)}" ixy="0" ixz="0"
+                    iyy="${(m/12) * (3*r*r + l*l)}" iyz="0"
+                    izz="${(m/2) * (r*r)}" />
+        </inertial>
+    </xacro:macro>
+    <xacro:macro name="sphere_inertia" params="m r o_xyz o_rpy">
+        <inertial>
+            <mass value="${m}" />
+            <origin xyz="${o_xyz}" rpy="${o_rpy}" />
+            <inertia ixx="${(2/5) * m * r * r}" ixy="0" ixz="0"
+                    iyy="${(2/5) * m * r * r}" iyz="0"
+                    izz="${(2/5) * m * r * r}" />
+        </inertial>
+    </xacro:macro>
+    <xacro:property name="base_length" value="0.6" />
+    <xacro:property name="base_width" value="0.4" />
+    <xacro:property name="base_height" value="0.2" />
+    <xacro:property name="wheel_radius" value="0.1" />
+    <xacro:property name="wheel_length" value="0.05" />
+    <link name="base_footprint" />
     <link name="base_link">
         <visual>
-            <origin xyz="0 0 0.06" />
             <geometry>
-                <box size="0.3 0.2 0.1" />
+                <box size="${base_length} ${base_width} ${base_height}" />
             </geometry>
+            <origin xyz="0 0 ${base_height / 2.0}" rpy="0 0 0" />
+            <material name="green" />
         </visual>
         <collision>
             <geometry>
-                <box size="0.3 0.2 0.1" />
+                <box size="${base_length} ${base_width} ${base_height}" />
             </geometry>
+            <origin xyz="0 0 ${base_height / 2.0}" rpy="0 0 0" />
         </collision>
-        <inertial>
-            <mass value="5.0" />
-            <inertia ixx="1.0" ixy="0.0" ixz="0.0" iyy="1.0" iyz="0.0" izz="1.0" />
-        </inertial>
+        <xacro:box_inertia m="5.0" x="${base_length}" y="${base_width}" z="${base_height}"
+                           o_xyz="0 0 ${base_height / 2.0}" o_rpy="0 0 0" />
     </link>
-    <link name="left_wheel_link">
+    <xacro:macro name="wheel_link" params="prefix">
+        <link name="${prefix}_wheel_link">
+            <visual>
+                <geometry>
+                    <cylinder radius="${wheel_radius}" length="${wheel_length}" />
+                </geometry>
+                <origin xyz="0 0 0" rpy="${pi / 2.0} 0 0" />
+                <material name="gray" />
+            </visual>
+            <collision>
+                <geometry>
+                    <sphere radius="${wheel_radius}" />
+                </geometry>
+                <origin xyz="0 0 0" rpy="0 0 0" />
+            </collision>
+            <xacro:cylinder_inertia m="1.0" r="${wheel_radius}" l="${wheel_length}"
+                                    o_xyz="0 0 0" o_rpy="${pi / 2.0} 0 0" />
+        </link>
+    </xacro:macro>
+    <xacro:wheel_link prefix="right" />
+    <xacro:wheel_link prefix="left" />
+    <link name="caster_wheel_link">
         <visual>
-            <origin rpy="1.5707 0 0" />
             <geometry>
-                <cylinder radius="0.05" length="0.04" />
+                <sphere radius="${wheel_radius / 2.0}" />
             </geometry>
+            <origin xyz="0 0 0" rpy="0 0 0" />
+            <material name="gray" />
         </visual>
         <collision>
-            <origin rpy="1.5707 0 0" />
             <geometry>
-                <cylinder radius="0.05" length="0.04" />
+                <sphere radius="${wheel_radius / 2.0}" />
             </geometry>
+            <origin xyz="0 0 0" rpy="0 0 0" />
         </collision>
-        <inertial>
-            <mass value="0.5" />
-            <inertia ixx="1.0" ixy="0.0" ixz="0.0" iyy="1.0" iyz="0.0" izz="1.0" />
-        </inertial>
+        <xacro:sphere_inertia m="0.5" r="${wheel_radius / 2.0}"
+                              o_xyz="0 0 0" o_rpy="0 0 0" />
     </link>
-    <link name="right_wheel_link">
-        <visual>
-            <origin rpy="1.5707 0 0" />
-            <geometry>
-                <cylinder radius="0.05" length="0.04" />
-            </geometry>
-        </visual>
-        <collision>
-            <origin rpy="1.5707 0 0" />
-            <geometry>
-                <cylinder radius="0.05" length="0.04" />
-            </geometry>
-        </collision>
-        <inertial>
-            <mass value="0.5" />
-            <inertia ixx="1.0" ixy="0.0" ixz="0.0" iyy="1.0" iyz="0.0" izz="1.0" />
-        </inertial>
-    </link>
-    <joint name="left_wheel_joint" type="continuous">
+    <joint name="base_joint" type="fixed">
+        <parent link="base_footprint" />
+        <child link="base_link" />
+        <origin xyz="0 0 ${wheel_radius}" rpy="0 0 0" />
+    </joint>
+    <joint name="base_right_wheel_joint" type="continuous">
+        <parent link="base_link" />
+        <child link="right_wheel_link" />
+        <origin xyz="${-base_length / 4.0} ${-(base_width + wheel_length) / 2.0} 0" rpy="0 0 0" />
+        <axis xyz="0 1 0" />
+    </joint>
+    <joint name="base_left_wheel_joint" type="continuous">
         <parent link="base_link" />
         <child link="left_wheel_link" />
-        <origin xyz="0 0.12 0.04" />
+        <origin xyz="${-base_length / 4.0} ${(base_width + wheel_length) / 2.0} 0" rpy="0 0 0" />
         <axis xyz="0 1 0" />
     </joint>
-    <joint name="right_wheel_joint" type="continuous">
+    <joint name="base_caster_wheel_joint" type="fixed">
         <parent link="base_link" />
-        <child link="right_wheel_link" />
-        <origin xyz="0 -0.12 0.04" />
-        <axis xyz="0 1 0" />
+        <child link="caster_wheel_link" />
+        <origin xyz="${base_length / 3.0} 0 ${-wheel_radius / 2.0}" rpy="0 0 0" />
     </joint>
-    <plugin
-        filename="gz-sim-diff-drive-system"
-        name="gz::sim::systems::DiffDrive">
-        <left_joint>left_wheel_joint</left_joint>
-        <right_joint>right_wheel_joint</right_joint>
-        <frame_id>odom</frame_id>
-        <child_frame_id>base_link</child_frame_id>
-        <wheel_separation>0.24</wheel_separation>
-        <wheel_radius>0.05</wheel_radius>
-    </plugin>
-    <plugin
-        filename="gz-sim-joint-state-publisher-system"
-        name="gz::sim::systems::JointStatePublisher">
-    </plugin>
+    <gazebo reference="caster_wheel_link">
+        <mu1 value="0.1" />
+        <mu2 value="0.1" />
+    </gazebo>
+    <gazebo>
+        <plugin
+            filename="gz-sim-diff-drive-system"
+            name="gz::sim::systems::DiffDrive">
+            <left_joint>base_left_wheel_joint</left_joint>
+            <right_joint>base_right_wheel_joint</right_joint>
+            <frame_id>odom</frame_id>
+            <child_frame_id>base_footprint</child_frame_id>
+            <wheel_separation>0.45</wheel_separation>
+            <wheel_radius>0.1</wheel_radius>
+        </plugin>
+    </gazebo>
+    <gazebo>
+        <plugin
+            filename="gz-sim-joint-state-publisher-system"
+            name="gz::sim::systems::JointStatePublisher">
+        </plugin>
+    </gazebo>
 </robot>

Commit message: Added a camera

File: src/line_follower_description/urdf/dummy_bot.urdf.xacro (robot description, xacro)
@@ -7,4 +7,7 @@
         <color rgba="0.7 0.7 0.7 1" />
     </material>
+    <material name="red">
+        <color rgba="0.6 0 0 1" />
+    </material>
     <xacro:macro name="box_inertia" params="m x y z o_xyz o_rpy">
         <inertial>
@@ -12,6 +15,6 @@
             <origin xyz="${o_xyz}" rpy="${o_rpy}" />
             <inertia ixx="${(m/12) * (z*z + y*y)}" ixy="0" ixz="0"
-                    iyy="${(m/12) * (x*x + z*z)}" iyz="0"
-                    izz="${(m/12) * (x*x + y*y)}" />
+                iyy="${(m/12) * (x*x + z*z)}" iyz="0"
+                izz="${(m/12) * (x*x + y*y)}" />
         </inertial>
     </xacro:macro>
@@ -21,6 +24,6 @@
             <origin xyz="${o_xyz}" rpy="${o_rpy}" />
             <inertia ixx="${(m/12) * (3*r*r + l*l)}" ixy="0" ixz="0"
-                    iyy="${(m/12) * (3*r*r + l*l)}" iyz="0"
-                    izz="${(m/2) * (r*r)}" />
+                iyy="${(m/12) * (3*r*r + l*l)}" iyz="0"
+                izz="${(m/2) * (r*r)}" />
         </inertial>
     </xacro:macro>
@@ -30,6 +33,6 @@
             <origin xyz="${o_xyz}" rpy="${o_rpy}" />
             <inertia ixx="${(2/5) * m * r * r}" ixy="0" ixz="0"
-                    iyy="${(2/5) * m * r * r}" iyz="0"
-                    izz="${(2/5) * m * r * r}" />
+                iyy="${(2/5) * m * r * r}" iyz="0"
+                izz="${(2/5) * m * r * r}" />
         </inertial>
     </xacro:macro>
@@ -46,5 +49,5 @@
             </geometry>
             <origin xyz="0 0 ${base_height / 2.0}" rpy="0 0 0" />
-            <material name="green" />
+            <material name="red" />
         </visual>
         <collision>
@@ -55,5 +58,5 @@
         </collision>
         <xacro:box_inertia m="5.0" x="${base_length}" y="${base_width}" z="${base_height}"
-                           o_xyz="0 0 ${base_height / 2.0}" o_rpy="0 0 0" />
+            o_xyz="0 0 ${base_height / 2.0}" o_rpy="0 0 0" />
     </link>
     <xacro:macro name="wheel_link" params="prefix">
@@ -73,5 +76,5 @@
             </collision>
             <xacro:cylinder_inertia m="1.0" r="${wheel_radius}" l="${wheel_length}"
-                                    o_xyz="0 0 0" o_rpy="${pi / 2.0} 0 0" />
+                o_xyz="0 0 0" o_rpy="${pi / 2.0} 0 0" />
         </link>
     </xacro:macro>
@@ -93,5 +96,5 @@
         </collision>
         <xacro:sphere_inertia m="0.5" r="${wheel_radius / 2.0}"
-                              o_xyz="0 0 0" o_rpy="0 0 0" />
+            o_xyz="0 0 0" o_rpy="0 0 0" />
     </link>
     <joint name="base_joint" type="fixed">
@@ -139,3 +142,43 @@
         </plugin>
     </gazebo>
+    <!-- Camera -->
+    <link name="camera_link">
+        <visual>
+            <geometry>
+                <box size="0.05 0.05 0.05" />
+            </geometry>
+            <material name="green" />
+        </visual>
+        <collision>
+            <geometry>
+                <box size="0.05 0.05 0.05" />
+            </geometry>
+        </collision>
+        <inertial>
+            <mass value="0.1" />
+            <inertia ixx="0.0001" iyy="0.0001" izz="0.0001"
+                ixy="0.0" ixz="0.0" iyz="0.0" />
+        </inertial>
+    </link>
+    <joint name="camera_joint" type="fixed">
+        <parent link="base_link" />
+        <child link="camera_link" />
+        <origin xyz="0.3 0 ${base_height + 0.05}" rpy="0 0 0" />
+    </joint>
+    <gazebo>
+        <plugin filename="gz-sim-sensors-system"
+            name="gz::sim::systems::Sensors">
+            <sensor>
+                <camera>
+                    <image_topic>/camera/image_raw</image_topic>
+                    <depth_topic>/camera/depth_raw</depth_topic>
+                    <fov>1.047</fov> <!-- 60 degrees -->
+                    <width>640</width>
+                    <height>480</height>
+                    <update_rate>30</update_rate>
+                    <link>camera_link</link>
+                </camera>
+            </sensor>
+        </plugin>
+    </gazebo>
 </robot>

Commit message: Few bug fixes

File: src/line_follower_description/urdf/dummy_bot.urdf.xacro (robot description, xacro)
@@ -164,21 +164,25 @@
         <parent link="base_link" />
         <child link="camera_link" />
-        <origin xyz="0.3 0 ${base_height + 0.05}" rpy="0 0 0" />
+        <origin xyz="0.3 0 ${base_height}" rpy="0 0 0" />
     </joint>
-    <gazebo>
-        <plugin filename="gz-sim-sensors-system"
-            name="gz::sim::systems::Sensors">
-            <sensor>
-                <camera>
-                    <image_topic>/camera/image_raw</image_topic>
-                    <depth_topic>/camera/depth_raw</depth_topic>
-                    <fov>1.047</fov> <!-- 60 degrees -->
+    <gazebo reference="camera_link">
+        <sensor name="camera_sensor" type="camera">
+            <update_rate>30</update_rate>
+            <camera>
+                <horizontal_fov>1.047</horizontal_fov>
+                <image>
                     <width>640</width>
                     <height>480</height>
-                    <update_rate>30</update_rate>
-                    <link>camera_link</link>
-                </camera>
-            </sensor>
-        </plugin>
+                    <format>R8G8B8</format>
+                </image>
+                <clip>
+                    <near>0.1</near>
+                    <far>100.0</far>
+                </clip>
+            </camera>
+            <always_on>true</always_on>
+            <visualize>true</visualize>
+            <topic>/camera/image_raw</topic>
+        </sensor>
     </gazebo>
 </robot>

Commit message: Removed temp files

File: src/line_follower_description/urdf/dummy_bot.urdf.xacro (robot description, xacro)
@@ -164,5 +164,5 @@
         <parent link="base_link" />
         <child link="camera_link" />
-        <origin xyz="0.3 0 ${base_height}" rpy="0 0 0" />
+        <origin xyz="0.3 0 ${base_height / 4.0}" rpy="0 0 0" />
     </joint>
     <gazebo reference="camera_link">

Commit message: A camera node split into two.

File: src/line_follower_description/urdf/dummy_bot.urdf.xacro (robot description, xacro)
@@ -164,5 +164,5 @@
         <parent link="base_link" />
         <child link="camera_link" />
-        <origin xyz="0.3 0 ${base_height / 4.0}" rpy="0 0 0" />
+        <origin xyz="0.3 0 ${base_height}" rpy="0 0.785 0" />
     </joint>
     <gazebo reference="camera_link">
@@ -170,13 +170,13 @@
             <update_rate>30</update_rate>
             <camera>
-                <horizontal_fov>1.047</horizontal_fov>
+                <horizontal_fov>0.70</horizontal_fov>
                 <image>
-                    <width>1980</width>
-                    <height>1080</height>
+                    <width>990</width>
+                    <height>540</height>
                     <format>R8G8B8</format>
                 </image>
                 <clip>
                     <near>0.1</near>
-                    <far>100.0</far>
+                    <far>10.0</far>
                 </clip>
             </camera>

Commit message: Added a new camera

File: src/line_follower_description/urdf/dummy_bot.urdf.xacro (robot description, xacro)
@@ -164,5 +164,5 @@
         <parent link="base_link" />
         <child link="camera_link" />
-        <origin xyz="0.3 0 ${base_height}" rpy="0 0.785 0" />
+        <origin xyz="0.3 0 ${base_height}" rpy="0 0.35 0" />
     </joint>
     <gazebo reference="camera_link">
@@ -186,3 +186,47 @@
         </sensor>
     </gazebo>
+    <!-- Camera 2 -->
+    <link name="camera_link2">
+        <visual>
+            <geometry>
+                <box size="0.05 0.05 0.05" />
+            </geometry>
+            <material name="green" />
+        </visual>
+        <collision>
+            <geometry>
+                <box size="0.05 0.05 0.05" />
+            </geometry>
+        </collision>
+        <inertial>
+            <mass value="0.1" />
+            <inertia ixx="0.0001" iyy="0.0001" izz="0.0001"
+                ixy="0.0" ixz="0.0" iyz="0.0" />
+        </inertial>
+    </link>
+    <joint name="camera_joint2" type="fixed">
+        <parent link="base_link" />
+        <child link="camera_link2" />
+        <origin xyz="0.3 0 ${base_height / 4.0}" rpy="0 0 0" />
+    </joint>
+    <gazebo reference="camera_link2">
+        <sensor name="camera_sensor2" type="camera">
+            <update_rate>30</update_rate>
+            <camera>
+                <horizontal_fov>1.047</horizontal_fov>
+                <image>
+                    <width>990</width>
+                    <height>540</height>
+                    <format>R8G8B8</format>
+                </image>
+                <clip>
+                    <near>0.1</near>
+                    <far>100.0</far>
+                </clip>
+            </camera>
+            <always_on>1</always_on>
+            <visualize>true</visualize>
+            <topic>/visuals</topic>
+        </sensor>
+    </gazebo>
 </robot>

Commit message: few fixes

File: src/line_follower_description/urdf/dummy_bot.urdf.xacro (robot description, xacro)
@@ -37,5 +37,5 @@
         </inertial>
     </xacro:macro>
-    <xacro:property name="base_length" value="0.6" />
+    <xacro:property name="base_length" value="0.2" />
     <xacro:property name="base_width" value="0.4" />
     <xacro:property name="base_height" value="0.2" />
@@ -164,5 +164,5 @@
         <parent link="base_link" />
         <child link="camera_link" />
-        <origin xyz="0.3 0 ${base_height}" rpy="0 0.35 0" />
+        <origin xyz="${base_length / 2.0} 0 ${base_height}" rpy="0 0.35 0" />
     </joint>
     <gazebo reference="camera_link">
@@ -208,5 +208,5 @@
         <parent link="base_link" />
         <child link="camera_link2" />
-        <origin xyz="0.3 0 ${base_height / 4.0}" rpy="0 0 0" />
+        <origin xyz="${base_length / 2.0} 0 ${base_height / 4.0}" rpy="0 0 0" />
     </joint>
     <gazebo reference="camera_link2">

Commit message: using quat

File: src/line_follower_description/urdf/dummy_bot.urdf.xacro (robot description, xacro)
@@ -37,5 +37,5 @@
         </inertial>
     </xacro:macro>
-    <xacro:property name="base_length" value="0.2" />
+    <xacro:property name="base_length" value="0.4" />
     <xacro:property name="base_width" value="0.4" />
     <xacro:property name="base_height" value="0.2" />
